File: GeigerCounter.sch (EAGLE design)
At the start: 40 parts, among them IC1 TLC555CP, IC2 ATtiny2313A-SU, J1 LND 712, J2 I2C, J3 ICSP, J4 I/O, Q1 STN83003, Q2 MMBT2222ALT3G, Q3 MMBT2222ALT3G, Q4 8 MHz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

Commit message: silkscreen tweaks
Parts:
- removed J4: I/O, freetronics-master-v1:M05PTH
- added Q6: SMD Buzzer, freetronics-master-v1:BUZZERSMD12X12
- J1: value LND 712 -> I2C; device SparkFun:GEIGER_TUBELND712 -> freetronics-master-v1:M04PTH
- J2: value I2C -> ICSP; device freetronics-master-v1:M04PTH -> connectors:ICSP-6; VALUE (none) -> ICSP
- J3: value ICSP -> I/O; device connectors:ICSP-6 -> freetronics-master-v1:M05PTH; VALUE ICSP -> (none)
- Q1: value STN83003 -> LND 712; device transistor-neu-to92:-NPN-SOT223 -> SparkFun:GEIGER_TUBELND712; PACKAGE SOT-223 -> (none)
- Q2: value MMBT2222ALT3G -> STN83003; device SparkFun:TRANSISTOR_NPNSOT23 -> transistor-neu-to92:-NPN-SOT223; PACKAGE SOT23-3 -> SOT-223
- Q4: value 8 MHz -> MMBT2222ALT3G; device freetronics-master-v1:CRYSTALHC49US -> SparkFun:TRANSISTOR_NPNSOT23; PACKAGE HC-49US -> SOT23-3
- Q5: value SMD Buzzer -> 8 MHz; device freetronics-master-v1:BUZZERSMD12X12 -> freetronics-master-v1:CRYSTALHC49US; PACKAGE (none) -> HC-49US
- R9: value 100kΩ -> 100k
- renumbered S to S1
Connections:
- net !RESET: now also J2.5; no longer J3.5
- net +3V3: now also J1.1, J2.2, J3.1; no longer J2.1, J3.2, J4.1
- net GM_PULSE: now also Q3.C; no longer Q2.C
- net GND: now also J1.2, J2.6, J3.2, Q4.E, Q6.GND; no longer J2.2, J3.6, J4.2, Q2.E, Q5.GND
- net N$1: now also Q1.VCC; no longer J1.VCC
- net N$14: now also Q2.B; no longer Q1.B
- net N$15: now also Q4.C; no longer Q3.C
- net N$26: now also J3.3; no longer J4.3
- net N$27: now also J3.4; no longer J4.4
- net N$28: now also Q5.1; no longer Q4.1
- net N$29: now also Q5.2; no longer Q4.2
- net N$31: now also J2.1; no longer J3.1
- net N$35: now also Q6.POS; no longer Q5.POS
- net N$48: now also Q1.GND; no longer J1.GND
- net N$49: now also Q3.B; no longer Q2.B
- net N$55: now also Q2.E, Q4.B; no longer Q1.E, Q3.B
- net N$57: now also Q2.C; no longer Q1.C
- net PULSE: now also J3.5; no longer J4.5
- net SCL: now also J1.4, J2.3; no longer J2.4, J3.3
- net SDA: now also J1.3, J2.4; no longer J2.3, J3.4
Other:
- moved on the sheet: Q2, Q3
